File: schematics/LED_Device/LED_Device.kicad_sch (KiCad schematic)
At the start: 3 parts, among them U1 ESP32S-WROOM-32, U2 MAX98357A

Commit message: Updated Schematic Drawings
Schematics have been updated to the current build status of the project.
Parts:
- removed LS1: Speaker, symbol Device:Speaker
- removed U2: MAX98357A, symbol 1A-AudioDRV_sym:MAX98357A
- added D1: LED STRIP, symbol Device:LED_Series_Pad
- added SW1, SW2, SW3: SW_Push_Dual, symbol Switch:SW_Push_Dual
- added U2: Oiyagai Breadboard Power Module, Package_TO_SOT_SMD:TO-252-2, symbol Regulator_Linear:KA78M05_TO252
- added U3: ~, symbol 1A-Power:AXLHNITI
Connections:
- net +3V3 is gone; now on net GNDREF: U1. (Tx)
- net GNDREF: now also D1.2 (A), SW1.4, SW2.4, SW3.4, U2.2 (GND), U3. (Vout)
- new net: SW1.1, U1. (Tx)
- new net: SW3.1, U1. (Tx)
- new net: SW2.1, U1. (Tx)
- new net: D1.1 (K), U1. (Tx), U2.3 (VO)
- new net: D1.3 (PAD), U1. (Tx)
- new net: U2.1 (VI), U3. (Vout)
- new net +12V: U3. (Vout)
Other:
- note added: "5V"
- note added: "GND"
- note added: "SIGNAL"
- note added: "Type B USA Socket"
- note removed: "Circuit for MAX98357A"
- title: ESP32S Based Speaker using MAX98357A -> ESP32S Based LED Controller
